Commit message: Added Collisions to Drone

File: navigation/models/scout/scout.gazebo.xacro (robot description, xacro)
@@ -81,4 +81,22 @@
     </plugin>
   </gazebo>
+<gazebo reference="base_link">
+  <self_collide>false</self_collide>
+  <surface>
+    <contact>
+      <!-- default mask: collide with world -->
+      <collide_bitmask>0xFFFF</collide_bitmask>
+    </contact>
+    <friction>
+      <ode>
+        <mu>0.8</mu>
+        <mu2>0.6</mu2>
+      </ode>
+    </friction>
+    <bounce>
+      <restitution_coefficient>0.05</restitution_coefficient>
+    </bounce>
+  </surface>
+</gazebo>
   <!-- Publish odometry separately -->
 <gazebo>

File: navigation/models/scout/scout.urdf.xacro (robot description, xacro)
@@ -9,47 +9,49 @@
   <!-- Main link -->
   <link name="base_link">
-    <inertial>
-      <origin xyz="0 0 0" rpy="0 0 0"/>
-      <mass value="0.503"/> <!-- kg -->
-      <inertia ixx="1.805e-3" ixy="-8.619e-7" ixz="1.555e-5"
-               iyy="1.764e-3" iyz="3.595e-7"
-               izz="3.328e-3" />
-    </inertial>
-<!--     <collision name="collision">
-      <origin xyz="-0.00424 0.00014 -0.00595" rpy="0 0 0"/>
-      <geometry>
-        <box size="0.5 0.5 0.2"/>
-      </geometry>
-    </collision> -->
-    <visual name="hull">
-      <geometry>
-        <mesh filename="file://$(find navigation)/models/scout/meshes/hull.dae"/>
-      </geometry>
-    </visual>
-    <visual name="propeller_rr">
-      <origin xyz="-0.09035 -0.11423 -0.00501" rpy="0 0 0"/>
-      <geometry>
-        <mesh filename="file://$(find navigation)/models/scout/meshes/propeller_rr.dae"/>
-      </geometry>
-    </visual>
-    <visual name="propeller_rl">
-      <origin xyz="0.09035 0.11452 -0.00501" rpy="0 0 0"/>
-      <geometry>
-        <mesh filename="file://$(find navigation)/models/scout/meshes/propeller_rl.dae"/>
-      </geometry>
-    </visual>
-    <visual name="propeller_fr">
-      <origin xyz="0.08456 -0.11435 -0.00501" rpy="0 0 0"/>
-      <geometry>
-        <mesh filename="file://$(find navigation)/models/scout/meshes/propeller_fr.dae"/>
-      </geometry>
-    </visual>
-    <visual name="propeller_fl">
-      <origin xyz="0.08456 0.11463 -0.00501" rpy="0 0 0"/>
-      <geometry>
-        <mesh filename="file://$(find navigation)/models/scout/meshes/propeller_fl.dae"/>
-      </geometry>
-    </visual>
-  </link>
+  <inertial>
+    <origin xyz="0 0 0" rpy="0 0 0"/>
+    <mass value="0.503"/> <!-- kg -->
+    <inertia ixx="1.805e-3" ixy="-8.619e-7" ixz="1.555e-5"
+             iyy="1.764e-3" iyz="3.595e-7"
+             izz="3.328e-3" />
+  </inertial>
+  <!-- COLLISION: matches your SDF body collision -->
+  <collision name="base_link_collision">
+    <origin xyz="-0.00424 0.00014 -0.00595" rpy="0 0 0"/>
+    <geometry>
+      <box size="0.316618 0.330564 0.089582"/>
+    </geometry>
+  </collision>
+  <!-- Visuals (unchanged) -->
+  <visual name="hull">
+    <geometry>
+      <mesh filename="file://$(find navigation)/models/scout/meshes/hull.dae"/>
+    </geometry>
+  </visual>
+  <visual name="propeller_rr">
+    <origin xyz="-0.09035 -0.11423 -0.00501" rpy="0 0 0"/>
+    <geometry>
+      <mesh filename="file://$(find navigation)/models/scout/meshes/propeller_rr.dae"/>
+    </geometry>
+  </visual>
+  <visual name="propeller_rl">
+    <origin xyz="0.09035 0.11452 -0.00501" rpy="0 0 0"/>
+    <geometry>
+      <mesh filename="file://$(find navigation)/models/scout/meshes/propeller_rl.dae"/>
+    </geometry>
+  </visual>
+  <visual name="propeller_fr">
+    <origin xyz="0.08456 -0.11435 -0.00501" rpy="0 0 0"/>
+    <geometry>
+      <mesh filename="file://$(find navigation)/models/scout/meshes/propeller_fr.dae"/>
+    </geometry>
+  </visual>
+  <visual name="propeller_fl">
+    <origin xyz="0.08456 0.11463 -0.00501" rpy="0 0 0"/>
+    <geometry>
+      <mesh filename="file://$(find navigation)/models/scout/meshes/propeller_fl.dae"/>
+    </geometry>
+  </visual>
+</link>
   <joint name="imu_joint" type="fixed">
     <parent link="base_link"/>

Commit message: aded thermal camera to drone, added thermal detection scripts

File: navigation/models/scout/scout.gazebo.xacro (robot description, xacro)
@@ -1,3 +1,3 @@
-<?xml version="1.0"?>
+ <?xml version="1.0"?>
 <robot name="scout" xmlns:xacro="http://ros.org/wiki/xacro">
   <xacro:arg name="laser_visual"  default="false" />
@@ -189,4 +189,36 @@
       <gz_frame_id>camera_link</gz_frame_id>
     </sensor>
+     <!-- ==================== Thermal Camera Sensor ==================== -->
+  <sensor name="thermal_camera" type="thermal">
+    <always_on>true</always_on>
+    <update_rate>10</update_rate>
+    <visualize>$(arg camera_visual)</visualize>
+    <pose>0 0 0 0 0 0</pose>
+    <camera>
+      <!-- Approx 60 deg field of view -->
+      <horizontal_fov>1.047</horizontal_fov>
+      <image>
+        <width>640</width>
+        <height>480</height>
+        <!-- Thermal cameras output 16-bit grayscale (Kelvin values) -->
+        <format>L16</format>
+      </image>
+      <clip>
+        <near>0.2</near>
+        <far>50</far>
+      </clip>
+    </camera>
+    <!-- Thermal parameters -->
+    <thermal_camera>
+      <min_temperature>273.15</min_temperature>   <!-- 0°C -->
+      <max_temperature>373.15</max_temperature>   <!-- 100°C -->
+      <resolution>0.1</resolution>                <!-- Temperature resolution in K -->
+    </thermal_camera>
+    <!-- Topics for Gazebo transport (bridge these to ROS) -->
+    <topic>/model/scout/thermal/image</topic>
+    <camera_info_topic>/model/scout/thermal/camera_info</camera_info_topic>
+    <!-- If you use TF optical frames for cameras, uncomment and point to it -->
+    <!-- <gz_frame_id>camera_thermal_optical_frame</gz_frame_id> -->
+  </sensor>
   </gazebo>
 </robot>

File: navigation/models/scout/scout.urdf.xacro (robot description, xacro)
@@ -127,3 +127,18 @@
   </joint>
   <link name="camera_depth_optical_frame"/>
+  <!-- Thermal camera frames -->
+  <joint name="camera_thermal_joint" type="fixed">
+    <!-- Re-use the same position as RGB by default; tweak as needed -->
+    <origin xyz="${r200_cam_rgb_px} ${r200_cam_rgb_py} ${r200_cam_rgb_pz}" rpy="0 0 0"/>
+    <parent link="camera_link"/>
+    <child link="camera_thermal_frame"/>
+  </joint>
+  <link name="camera_thermal_frame"/>
+  <joint name="camera_thermal_optical_joint" type="fixed">
+    <!-- Standard optical frame rotation: X forward, Z down -->
+    <origin xyz="0 0 0" rpy="-1.57 0 -1.57"/>
+    <parent link="camera_thermal_frame"/>
+    <child link="camera_thermal_optical_frame"/>
+  </joint>
+  <link name="camera_thermal_optical_frame"/>
 </robot>

Commit message: thirdperson camera, gui adjustments

File: navigation/models/scout/scout.gazebo.xacro (robot description, xacro)
@@ -3,4 +3,5 @@
   <xacro:arg name="laser_visual"  default="true"/>
   <xacro:arg name="camera_visual" default="true"/>
+  <xacro:arg name="third_person" default="true"/>
   <xacro:arg name="imu_visual"    default="true"/>
   <!-- <xacro:include filename="$(find 41068_ignition_bringup)/urdf/wheel.urdf.xacro"/> -->
@@ -209,5 +210,5 @@
         <clip>
           <near>0.1</near>
-          <far>40</far>
+          <far>200</far>
         </clip>
         <!-- depth_camera near/far clip seems to be ignored for some reason -->
@@ -232,3 +233,36 @@
     </sensor>
   </gazebo>
+  <gazebo reference="third_person_link">
+    <sensor name="third_person" type="camera">
+      <camera>
+        <horizontal_fov>2.0944</horizontal_fov>
+        <image>
+          <width>720</width>
+          <height>480</height>
+        </image>
+        <clip>
+          <near>0.1</near>
+          <far>200</far>
+        </clip>
+        <!-- depth_camera near/far clip seems to be ignored for some reason -->
+        <!--    We're using Ignition Gazebo Fortress, which uses sdf format 1.9: http://sdformat.org/tutorials?tut=roadmap -->
+        <!--    This takes the depth_camera parameter with near / far clip http://sdformat.org/spec?ver=1.4&elem=sensor  -->
+        <!-- We also use ign sensors v6 ( run ls | grep libignition-sensors in /usr/lib/x86_64-linux-gnu)-->
+        <!-- Looking at the source code, the sdf sets HasDepthCamera() and corresponding HasDepthNearClip() & HasDepthFarClip() which are used in RgbdCameraSensor.cc, so this should work? -->
+        <!--    SDF description of Camera: https://github.com/gazebosim/sdformat/blob/sdf9/src/Camera.cc#L598-->
+        <!--    Camera sensor source code: https://github.com/gazebosim/gz-sensors/blob/ign-sensors6/src/RgbdCameraSensor.cc#L311  -->
+        <!--<depth_camera>
+          <clip>
+            <near>0.4</near>
+            <far>10</far>
+          </clip>
+        </depth_camera>-->
+      </camera>
+      <always_on>1</always_on>
+      <update_rate>3</update_rate> <!--10-->
+      <visualize>$(arg third_person)</visualize>
+      <topic>/model/scout/third_person</topic>
+      <gz_frame_id>third_person_link</gz_frame_id>
+    </sensor>
+  </gazebo>
 </robot>

File: navigation/models/scout/scout.urdf.xacro (robot description, xacro)
@@ -86,4 +86,12 @@
     <child link="camera_link"/>
   </joint>
+  <joint name="third_person_joint" type="fixed">
+    <parent link="base_link"/>
+    <child link="third_person_link"/>
+    <origin xyz="-0.25 0.0 0.25" rpy="0 0.785398 0"/> <!-- 0.5 0.0 0.9 -->
+  </joint>
+  <link name="third_person_link" type="fixed">
+    <origin xyz="0.0 0.0 0.0" rpy="0 0 0"/> <!-- 0.5 0.0 0.9 -->
+  </link>
   <link name="camera_link">
     <visual>
