Commit message: Camera

File: navigation/models/scout/scout.urdf.xacro (robot description, xacro)
@@ -85,4 +85,5 @@
     <parent link="base_link"/>
     <child link="camera_link"/>
+    <origin xyz="0.2 0 1.1" rpy="0 0 0"/>
   </joint>
   <link name="camera_link">

Commit message: Working on SLam making progress

File: navigation/models/scout/scout.urdf.xacro (robot description, xacro)
@@ -73,6 +73,12 @@
       <material name="dark"/>
     </visual>
+ <collision>
+    <origin xyz="0 0 0" rpy="0 0 0"/>
+    <geometry>
+      <cylinder length="0.04" radius="0.09"/>
+    </geometry>
+  </collision>
     <inertial>
-      <mass value="0" />
+      <mass value="0.1" />
       <origin xyz="0 0 0" />
       <inertia ixx="0.001" ixy="0.0" ixz="0.0"
